File: test/RoverMuxJig.sch (EAGLE design)
At the start: 22 parts, among them J1 ISP, Q1 16MHz, U1 ATMEGA328P_TQFP

Commit message: Updated jig
Parts:
- removed U$4: USB-MINIB-5PIN, SparkFun-Connectors:USB-MINIB-5PIN
- added C1: 104, rcl:C-USC0603
- added JP1: FTDI, SparkFun-Connectors:FTDI_BASICPTH
Connections:
- new net N$4: C1.1, JP1.1
- new net RX<: JP1.3, U1.PD0(RXD)
- new net TX>: JP1.2, U1.PD1(TXD)
- net !RESET: now also C1.2
- net 5V: now also JP1.4; no longer U$4.VBUS
- net GND: now also JP1.6; no longer U$4.GND
Changed lines of the file:
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@@
 <part name="J1" library="bt_avr" deviceset="AVRISP6" device="" value="ISP"/>
 <part name="GND3" library="mes" deviceset="GND" device=""/>
-<part name="U$4" library="SparkFun-Connectors" deviceset="USB-MINIB" device="-5PIN"/>
 <part name="U1" library="SparkFun-DigitalIC" deviceset="ATMEGA328P_TQFP" device="" value="ATMEGA328P_TQFP"/>
 <part name="R1" library="rcl" deviceset="R-US_" device="R0603" value="10K">
@@
 <part name="U$6" library="bt" deviceset="5V" device=""/>
 <part name="U$5" library="bt" deviceset="5V" device=""/>
+<part name="JP1" library="SparkFun-Connectors" deviceset="FTDI_BASIC" device="PTH" value="FTDI"/>
+<part name="U$7" library="bt" deviceset="5V" device=""/>
+<part name="GND7" library="mes" deviceset="GND" device=""/>
+<part name="C1" library="rcl" deviceset="C-US" device="C0603" value="104">
+<attribute name="PARTNO" value="C1608X7R1E104K080AA"/>
+</part>
 </parts>
 <sheets>
@@
 <instance part="J1" gate="A" x="35.56" y="154.94"/>
 <instance part="GND3" gate="1" x="17.78" y="154.94"/>
-<instance part="U$4" gate="G$1" x="228.6" y="63.5"/>
 <instance part="U1" gate="U$1" x="149.86" y="124.46"/>
 <instance part="R1" gate="G$1" x="109.22" y="154.94">
@@
 <instance part="U$6" gate="G$1" x="33.02" y="116.84"/>
 <instance part="U$5" gate="G$1" x="17.78" y="167.64"/>
+<instance part="JP1" gate="G$1" x="144.78" y="63.5" rot="MR0"/>
+<instance part="U$7" gate="G$1" x="134.62" y="81.28"/>
+<instance part="GND7" gate="1" x="137.16" y="50.8"/>
+<instance part="C1" gate="G$1" x="129.54" y="58.42" rot="R270">
+<attribute name="PARTNO" x="129.54" y="58.42" size="1.778" layer="96" rot="R270" display="off"/>
+</instance>
 </instances>
 <busses>
@@
 <pinref part="R1" gate="G$1" pin="2"/>
 <label x="114.3" y="154.94" size="1.778" layer="95"/>
+</segment>
+<segment>
+<pinref part="C1" gate="G$1" pin="2"/>
+<wire x1="124.46" y1="58.42" x2="111.76" y2="58.42" width="0.1524" layer="91"/>
+<label x="111.76" y="58.42" size="1.778" layer="95"/>
 </segment>
 </net>
@@
 <pinref part="GND4" gate="1" pin="GND"/>
 <pinref part="C10" gate="G$1" pin="2"/>
-<wire x1="203.2" y1="66.04" x2="203.2" y2="50.8" width="0.1524" layer="91"/>
-<pinref part="U$4" gate="G$1" pin="GND"/>
-<wire x1="226.06" y1="63.5" x2="215.9" y2="63.5" width="0.1524" layer="91"/>
-<wire x1="215.9" y1="63.5" x2="215.9" y2="50.8" width="0.1524" layer="91"/>
-<wire x1="215.9" y1="50.8" x2="203.2" y2="50.8" width="0.1524" layer="91"/>
-<junction x="203.2" y="50.8"/>
-<wire x1="203.2" y1="50.8" x2="203.2" y2="48.26" width="0.1524" layer="91"/>
+<wire x1="203.2" y1="66.04" x2="203.2" y2="48.26" width="0.1524" layer="91"/>
 </segment>
 <segment>
@@
 <junction x="114.3" y="99.06"/>
 </segment>
+<segment>
+<pinref part="JP1" gate="G$1" pin="6"/>
+<pinref part="GND7" gate="1" pin="GND"/>
+<wire x1="139.7" y1="71.12" x2="137.16" y2="71.12" width="0.1524" layer="91"/>
+<wire x1="137.16" y1="71.12" x2="137.16" y2="53.34" width="0.1524" layer="91"/>
+</segment>
 </net>
 <net name="CH2RX" class="0">
@@
 <net name="5V" class="0">
 <segment>
-<wire x1="203.2" y1="78.74" x2="203.2" y2="83.82" width="0.1524" layer="91"/>
-<wire x1="203.2" y1="83.82" x2="203.2" y2="88.9" width="0.1524" layer="91"/>
-<wire x1="203.2" y1="73.66" x2="203.2" y2="78.74" width="0.1524" layer="91"/>
+<wire x1="203.2" y1="73.66" x2="203.2" y2="83.82" width="0.1524" layer="91"/>
 <pinref part="C10" gate="G$1" pin="1"/>
-<junction x="203.2" y="78.74"/>
-<pinref part="U$4" gate="G$1" pin="VBUS"/>
-<wire x1="226.06" y1="73.66" x2="215.9" y2="73.66" width="0.1524" layer="91"/>
-<wire x1="215.9" y1="73.66" x2="215.9" y2="78.74" width="0.1524" layer="91"/>
-<wire x1="215.9" y1="78.74" x2="203.2" y2="78.74" width="0.1524" layer="91"/>
 <pinref part="U$1" gate="G$1" pin="5V"/>
-<junction x="203.2" y="83.82"/>
 </segment>
 <segment>
@@
 <pinref part="U$5" gate="G$1" pin="5V"/>
 </segment>
-</net>
+<segment>
+<pinref part="JP1" gate="G$1" pin="4"/>
+<pinref part="U$7" gate="G$1" pin="5V"/>
+<wire x1="139.7" y1="66.04" x2="134.62" y2="66.04" width="0.1524" layer="91"/>
+<wire x1="134.62" y1="66.04" x2="134.62" y2="78.74" width="0.1524" layer="91"/>
+</segment>
+</net>
+<net name="N$4" class="0">
+<segment>
+<pinref part="JP1" gate="G$1" pin="1"/>
+<wire x1="139.7" y1="58.42" x2="132.08" y2="58.42" width="0.1524" layer="91"/>
+<pinref part="C1" gate="G$1" pin="1"/>
+</segment>
+</net>
+<net name="RX&lt;" class="0">
+<segment>
+<pinref part="JP1" gate="G$1" pin="3"/>
+<wire x1="139.7" y1="63.5" x2="111.76" y2="63.5" width="0.1524" layer="91"/>
+<label x="111.76" y="63.5" size="1.778" layer="95"/>
+</segment>
+<segment>
+<pinref part="U1" gate="U$1" pin="PD0(RXD)"/>
+<wire x1="172.72" y1="132.08" x2="185.42" y2="132.08" width="0.1524" layer="91"/>
+<label x="185.42" y="132.08" size="1.778" layer="95" rot="MR0"/>
+</segment>
+</net>
+<net name="TX&gt;" class="0">
+<segment>
+<pinref part="JP1" gate="G$1" pin="2"/>
+<wire x1="139.7" y1="60.96" x2="111.76" y2="60.96" width="0.1524" layer="91"/>
+<label x="111.76" y="60.96" size="1.778" layer="95"/>
+</segment>
+<segment>
+<pinref part="U1" gate="U$1" pin="PD1(TXD)"/>
+<wire x1="172.72" y1="129.54" x2="185.42" y2="129.54" width="0.1524" layer="91"/>
+<label x="185.42" y="129.54" size="1.778" layer="95" rot="MR0"/>
+</segment>
+</net>
